File: Kernel.kicad_pcb (KiCad board)
At the start: 2 copper layers, 48.3 x 26.7 mm, 14 parts, among them J1 TTL, J2 L, J3 R, J4 Conn_01x02_Male, SW1 MODE, SW2 Reset, SW3 RePair, U1 ESP-12S

Commit message: update files
Other:
- board text added: "Flash"
- board text added: "Ver0.2"
- board text removed: "Upload"
- board text removed: "Ver0.1"
