File: 0_X/Kernel.kicad_pcb (KiCad board)
At the start: 2 copper layers, 48.3 x 26.7 mm, 14 parts, among them J1 TTL, J2 L, J3 R, J4 Conn_01x02_Male, SW1 MODE, SW2 Reset, SW3 RePair, U1 ESP-12S

Commit message: update Ver 1.1
Parts:
- J4: value Conn_01x02_Male -> TTL
